Commit message: autunomous-vehicle

File: ros_ws/src/simulation/racer_description/urdf/racer.xacro (robot description, xacro)
@@ -2,4 +2,51 @@
 <robot name="myrobot"
   xmlns:xacro="http://www.ros.org/wiki/xacro">
+  <gazebo>
+    <plugin filename="libgazebo_ros2_control.so" name="gazebo_ros2_control">
+      <robot_param>robot_description</robot_param>
+      <robot_param_node>robot_state_publisher</robot_param_node>
+      <parameters>/home/ty/f1test_ws/ar-tu-do/control_config.yaml</parameters>
+    </plugin>
+  </gazebo>
+  <!-- ROS2 Control Interfaces -->
+  <ros2_control name="GazeboSystem" type="system">
+    <hardware>
+      <plugin>gazebo_ros2_control/GazeboSystem</plugin>
+    </hardware>
+    <!-- Rear Wheel Drive Joints -->
+    <joint name="left_wheel_back_hinge">
+      <command_interface name="velocity">
+        <param name="min">-100</param>
+        <param name="max">100</param>
+      </command_interface>
+      <state_interface name="position"/>
+      <state_interface name="velocity"/>
+    </joint>
+    <joint name="right_wheel_back_hinge">
+      <command_interface name="velocity">
+        <param name="min">-100</param>
+        <param name="max">100</param>
+      </command_interface>
+      <state_interface name="position"/>
+      <state_interface name="velocity"/>
+    </joint>
+    <!-- Front Wheel Steering Joints -->
+    <joint name="left_steering_hinge">
+      <command_interface name="position">
+        <param name="min">-1.0</param>
+        <param name="max">1.0</param>
+      </command_interface>
+      <state_interface name="position"/>
+      <state_interface name="velocity"/>
+    </joint>
+    <joint name="right_steering_hinge">
+      <command_interface name="position">
+        <param name="min">-1.0</param>
+        <param name="max">1.0</param>
+      </command_interface>
+      <state_interface name="position"/>
+      <state_interface name="velocity"/>
+    </joint>
+  </ros2_control>
   <xacro:arg name="simulation" default="false"/>
   <xacro:if value="$(arg simulation)">
@@ -17,4 +64,17 @@
   <xacro:property name="bodySizeH" value="0.1"/>
   <xacro:property name="bodyMass" value="3.5"/>
+  <!-- Wheel properties -->
+  <xacro:property name="wheel_radius" value="0.05" />
+  <xacro:property name="wheel_height" value="0.045" />
+  <xacro:property name="wheel_mass" value="0.2" />
+  <xacro:property name="base_x_origin_to_wheel_origin" value="0.16" />
+  <xacro:property name="base_y_origin_to_wheel_origin" value="0.1055" />
+  <xacro:property name="base_z_origin_to_wheel_origin" value="0" />
+  <xacro:property name="base_x_sphere_origin_to_wheel_origin" value="0.000" />
+  <xacro:property name="base_y_sphere_origin_to_wheel_origin" value="0.001" />
+  <xacro:property name="base_z_sphere_origin_to_wheel_origin" value="0" />
+  <!-- Steering properties -->
+  <xacro:property name="steering_radius" value="0.01" />
+  <xacro:property name="steering_mass" value="0.07" />
   <link name="base_link" />
   <joint name="base_link_joint" type="fixed">
@@ -28,5 +88,5 @@
       <mass value="${bodyMass}"/>
       <origin xyz="0 0 ${wheel_height/2}" rpy=" 0 0 0"/>
-      <box_inertia m="${bodyMass}" l="${bodySizeL}" b="${bodySizeB}" h="${bodySizeH}" />
+      <xacro:box_inertia m="${bodyMass}" l="${bodySizeL}" b="${bodySizeB}" h="${bodySizeH}" />
     </inertial>
     <collision name='collision'>
@@ -39,8 +99,14 @@
       <origin xyz="0 0 0" rpy=" 0 0 0"/>
       <geometry>
-        <mesh filename="package://racer_description/meshes/car.dae"/>
-      </geometry>
-    </visual>
-  </link>
+        <mesh filename="file:///home/ty/f1test_ws/ar-tu-do/ros_ws/install/racer_description/share/racer_description/meshes/car.dae"/>
+      </geometry>
+      <material name="car_material">
+        <color rgba="1.0 0.5 0.0 1.0"/>
+      </material>
+    </visual>
+  </link>
+  <gazebo reference="chassis">
+    <material>Gazebo/Orange</material>
+  </gazebo>
   <joint name="base_body_joint" type="fixed">
     <origin xyz="0 0 0" rpy="0 0 0" />
@@ -52,16 +118,19 @@
       <origin xyz="0 0 0.05" rpy=" 0 0 0"/>
       <geometry>
-        <mesh filename="package://racer_description/meshes/body.dae"/>
-      </geometry>
-    </visual>
-  </link>
+        <mesh filename="file:///home/ty/f1test_ws/ar-tu-do/ros_ws/install/racer_description/share/racer_description/meshes/body.dae"/>
+      </geometry>
+    </visual>
+  </link>
+  <gazebo reference="body">
+    <material>Gazebo/Blue</material>
+  </gazebo>
     <!--  Wheels  -->
-  <wheel fb="front" lr="left" parent="left_steering" translateX="1" translateY="1" left="1" OffsetJointX= "${base_x_sphere_origin_to_wheel_origin}" OffsetJointY= "${base_y_sphere_origin_to_wheel_origin}" OffsetJointZ= "${base_z_sphere_origin_to_wheel_origin}" OffsetY="0.02" />
-  <wheel fb="front" lr="right" parent="right_steering" translateX="1" translateY="-1" left="0" OffsetJointX= "${base_x_sphere_origin_to_wheel_origin}" OffsetJointY= "${base_y_sphere_origin_to_wheel_origin}" OffsetJointZ= "${base_z_sphere_origin_to_wheel_origin}" OffsetY="-0.02" />
-  <wheel fb="back" lr="left" parent="chassis" translateX="-1" translateY="1" left="1" OffsetJointX= "${base_x_origin_to_wheel_origin}" OffsetJointY= "${base_y_origin_to_wheel_origin}" OffsetJointZ= "${base_z_origin_to_wheel_origin}" OffsetY="0.021" />
-  <wheel fb="back" lr="right" parent="chassis" translateX="-1" translateY="-1" left="0" OffsetJointX= "${base_x_origin_to_wheel_origin}" OffsetJointY= "${base_y_origin_to_wheel_origin}" OffsetJointZ= "${base_z_origin_to_wheel_origin}" OffsetY="-0.021" />
+  <xacro:wheel fb="front" lr="left" parent="left_steering" translateX="1" translateY="1" left="1" OffsetJointX= "${base_x_sphere_origin_to_wheel_origin}" OffsetJointY= "${base_y_sphere_origin_to_wheel_origin}" OffsetJointZ= "${base_z_sphere_origin_to_wheel_origin}" OffsetY="0.02" />
+  <xacro:wheel fb="front" lr="right" parent="right_steering" translateX="1" translateY="-1" left="0" OffsetJointX= "${base_x_sphere_origin_to_wheel_origin}" OffsetJointY= "${base_y_sphere_origin_to_wheel_origin}" OffsetJointZ= "${base_z_sphere_origin_to_wheel_origin}" OffsetY="-0.02" />
+  <xacro:wheel fb="back" lr="left" parent="chassis" translateX="-1" translateY="1" left="1" OffsetJointX= "${base_x_origin_to_wheel_origin}" OffsetJointY= "${base_y_origin_to_wheel_origin}" OffsetJointZ= "${base_z_origin_to_wheel_origin}" OffsetY="0.021" />
+  <xacro:wheel fb="back" lr="right" parent="chassis" translateX="-1" translateY="-1" left="0" OffsetJointX= "${base_x_origin_to_wheel_origin}" OffsetJointY= "${base_y_origin_to_wheel_origin}" OffsetJointZ= "${base_z_origin_to_wheel_origin}" OffsetY="-0.021" />
   <!-- Steering -->
-  <steering_hinge lr="left" parent="chassis" translateY="1" OffsetY="0.01" />
-  <steering_hinge lr="right" parent="chassis" translateY="-1" OffsetY="-0.01" />
+  <xacro:steering_hinge lr="left" parent="chassis" translateY="1" OffsetY="0.01" />
+  <xacro:steering_hinge lr="right" parent="chassis" translateY="-1" OffsetY="-0.01" />
   <!-- Camera -->
   <link name="camera">
@@ -69,5 +138,5 @@
       <mass value="${cameraMass}" />
       <origin xyz="0 0 ${wheel_height/2}" rpy="0 0 0"/>
-      <box_inertia m="${cameraMass}" l="${cameraSizeL}" b="${cameraSizeB}" h="${cameraSizeH}" />
+      <xacro:box_inertia m="${cameraMass}" l="${cameraSizeL}" b="${cameraSizeB}" h="${cameraSizeH}" />
     </inertial>
     <collision>
@@ -80,8 +149,11 @@
       <origin xyz="0 0 0" rpy="0 0 0"/>
       <geometry>
-        <mesh filename="package://racer_description/meshes/ZED.dae"/>
-      </geometry>
-    </visual>
-  </link>s
+        <mesh filename="file:///home/ty/f1test_ws/ar-tu-do/ros_ws/install/racer_description/share/racer_description/meshes/ZED.dae"/>
+      </geometry>
+    </visual>
+  </link>
+  <gazebo reference="camera">
+    <material>Gazebo/Red</material>
+  </gazebo>
   <joint name="camera_joint" type="fixed">
     <axis xyz="0 1 0" />
@@ -95,5 +167,5 @@
       <mass value="${hokuyoMass}" />
       <origin xyz="0 0 ${wheel_height/2}" rpy="0 0 0"/>
-      <box_inertia m="${hokuyoMass}" l="${hokuyoSize}" b="${hokuyoSize}" h="${hokuyoSize}" />
+      <xacro:box_inertia m="${hokuyoMass}" l="${hokuyoSize}" b="${hokuyoSize}" h="${hokuyoSize}" />
     </inertial>
     <collision>
@@ -106,8 +178,11 @@
       <origin xyz="0 0 ${wheel_height/2}" rpy="0 0 0"/>
       <geometry>
-        <mesh filename="package://racer_description/meshes/hokuyo.dae"/>
-      </geometry>
-    </visual>
-  </link>
+        <mesh filename="file:///home/ty/f1test_ws/ar-tu-do/ros_ws/install/racer_description/share/racer_description/meshes/hokuyo.dae"/>
+      </geometry>
+    </visual>
+  </link>
+  <gazebo reference="laser">
+    <material>Gazebo/Green</material>
+  </gazebo>
   <joint name="laser_joint" type="fixed">
     <axis xyz="0 1 0" />

File: ros_ws/src/simulation/racer_description/urdf/racer_macros.xacro (robot description, xacro)
@@ -2,19 +2,19 @@
 <robot name="racer_macros" xmlns:xacro="http://www.ros.org/wiki/xacro">
   <!-- Inertias -->
-  <macro name="cylinder_inertia" params="m r h">
+  <xacro:macro name="cylinder_inertia" params="m r h">
     <inertia  ixx="${m*(3*r*r+h*h)/12}" ixy = "0" ixz = "0"
               iyy="${m*(3*r*r+h*h)/12}" iyz = "0"
               izz="${m*r*r/2}" />
-  </macro>
-  <macro name="box_inertia" params="m l b h">
+  </xacro:macro>
+  <xacro:macro name="box_inertia" params="m l b h">
     <inertia  ixx="${m*(b*b+h*h)/12}" ixy = "0" ixz = "0"
               iyy="${m*(l*l+h*h)/12}" iyz = "0"
               izz="${m*(l*l+b*b)/12}" />
-  </macro>
-  <macro name="sphere_inertia" params="m r">
+  </xacro:macro>
+  <xacro:macro name="sphere_inertia" params="m r">
     <inertia  ixx="${2*m*(r*r)/3}" ixy = "0" ixz = "0"
               iyy="${2*m*(r*r)/3}" iyz = "0"
               izz="${2*m*(r*r)/3}" />
-  </macro>
+  </xacro:macro>
   <!-- Wheels -->
   <property name="wheel_radius" value="0.05" />
@@ -32,5 +32,5 @@
         <mass value="${wheel_mass}" />
         <origin xyz="0 ${OffsetY} 0" rpy="${90*pi/180} 0 0"/>
-        <cylinder_inertia  m="${wheel_mass}" r="${wheel_radius}" h="${wheel_height}" />
+        <xacro:cylinder_inertia  m="${wheel_mass}" r="${wheel_radius}" h="${wheel_height}" />
       </inertial>
       <collision>
@@ -43,8 +43,11 @@
         <origin xyz="0 ${OffsetY} 0" rpy="0 0 ${left*pi}" />
         <geometry>
-          <mesh filename="package://racer_description/meshes/wheel.dae"/>
+          <mesh filename="file:///home/ty/f1test_ws/ar-tu-do/ros_ws/install/racer_description/share/racer_description/meshes/wheel.dae"/>
         </geometry>
       </visual>
     </link>
+    <gazebo reference="${lr}_wheel_${fb}">
+      <material>Gazebo/Black</material>
+    </gazebo>
     <joint name="${lr}_wheel_${fb}_hinge" type="continuous">
       <parent link="${parent}"/>
@@ -78,5 +81,5 @@
         <mass value="${steering_mass}" />
         <origin xyz="0 0 0" rpy="0 0 0"/>
-        <sphere_inertia  m="${steering_mass}" r="${steering_radius}" />
+        <xacro:sphere_inertia  m="${steering_mass}" r="${steering_radius}" />
       </inertial>
       <visual>
